Commit message: switch to ros control
changed the urdf description to match with the current version of ros_control

File: pr2_description/urdf/base_v0/base.transmission.xacro (robot description, xacro)
@@ -6,16 +6,24 @@
   <!--  Caster wheel transmission   -->
   <xacro:macro name="pr2_wheel_transmission_v0" params="suffix parent reflect">
-    <transmission type="pr2_mechanism_model/SimpleTransmission" name="${parent}_${suffix}_wheel_trans">
-      <actuator name="${parent}_${suffix}_wheel_motor" />
-      <joint name="${parent}_${suffix}_wheel_joint" />
-      <mechanicalReduction>${reflect * 624/35 * 80/18}</mechanicalReduction>
+    <transmission  name="${parent}_${suffix}_wheel_trans">
+      <type>pr2_mechanism_model/SimpleTransmission</type>
+      <actuator name="${parent}_${suffix}_wheel_motor">
+        <mechanicalReduction>${reflect * 624/35 * 80/18}</mechanicalReduction>
+      </actuator>
+      <joint name="${parent}_${suffix}_wheel_joint">
+        <hardwareInterface>EffortJointInterface</hardwareInterface>
+      </joint>
     </transmission>
   </xacro:macro>
   <!-- Hub transmission only -->
   <xacro:macro name="pr2_caster_transmission_v0" params="suffix">
-    <transmission type="pr2_mechanism_model/SimpleTransmission" name="${suffix}_rotation_trans">
-      <actuator name="${suffix}_rotation_motor" />
-      <joint name="${suffix}_rotation_joint" />
-      <mechanicalReduction>${-1 * 624/35 * 80/18}</mechanicalReduction>
+    <transmission name="${suffix}_rotation_trans">
+      <type>pr2_mechanism_model/SimpleTransmission</type>
+      <actuator name="${suffix}_rotation_motor">
+        <mechanicalReduction>${-1 * 624/35 * 80/18}</mechanicalReduction>
+      </actuator>
+      <joint name="${suffix}_rotation_joint">
+        <hardwareInterface>EffortJointInterface</hardwareInterface>
+      </joint>
     </transmission>
   </xacro:macro>

File: pr2_description/urdf/forearm_v0/forearm.transmission.xacro (robot description, xacro)
@@ -6,7 +6,12 @@
   <xacro:macro name="pr2_forearm_transmission_v0" params="side">
     <!-- Wrist flex , Wrist roll -->
-    <transmission type="pr2_mechanism_model/WristTransmission" name="${side}_wrist_trans">
-      <rightActuator name="${side}_wrist_r_motor" mechanicalReduction="${624/35*54/16}"/>
-      <leftActuator name="${side}_wrist_l_motor"  mechanicalReduction="${624/35*54/16}"/>
+    <transmission name="${side}_wrist_trans">
+      <type>pr2_mechanism_model/WristTransmission</type>
+      <rightActuator name="${side}_wrist_r_motor">
+        <mechanicalReduction>{624/35*54/16}</mechanicalReduction>
+      </rightActuator>
+      <leftActuator name="${side}_wrist_l_motor">
+        <mechanicalReduction>{624/35*54/16}</mechanicalReduction>
+      </leftActuator>
       <flexJoint name="${side}_wrist_flex_joint"  mechanicalReduction="-1.0" />
       <rollJoint name="${side}_wrist_roll_joint"  mechanicalReduction="1.0" />

File: pr2_description/urdf/gripper_v0/gripper.transmission.xacro (robot description, xacro)
@@ -15,5 +15,7 @@
     <!-- Please refer to mechanism_model/src/pr2_gripper_transmission.cpp for implementation.-->
     <!-- gazebo_mimic_pid is for sim only.                                                   -->
-    <transmission type="pr2_mechanism_model/PR2GripperTransmission" name="${side}_gripper_trans" >
+<!--
+    <transmission name="${side}_gripper_trans" >
+      <type>pr2_mechanism_model/PR2GripperTransmission</type>
       <actuator       name="${side}_gripper_motor" />
       <gap_joint      name="${side}_gripper_joint"
@@ -29,19 +31,28 @@
                       b="${b}"
                       r="${r}"
-                      />
+                      >
+        <hardwareInterface>EffortJointInterface</hardwareInterface>
+      </gap_joint>
+-->
       <!-- if a gazebo joint exists as [l|r]_gripper_joint, use this tag to have
            gripper transmission apply torque directly to prismatic joint
            this should be the default behavior in diamondback, deprecating this flag -->
+<!--
       <use_simulated_gripper_joint/>
+-->
       <!-- set passive joint angles so things look nice in rviz -->
+<!--
       <passive_joint  name="${side}_gripper_l_finger_joint"     />
       <passive_joint  name="${side}_gripper_r_finger_joint"     />
       <passive_joint  name="${side}_gripper_r_finger_tip_joint" />
       <passive_joint  name="${side}_gripper_l_finger_tip_joint" />
+-->
       <!-- screw joint to capture gripper "dynamics" -->
+<!--
       <simulated_actuated_joint name="${side}_gripper_motor_screw_joint"
                                 passive_actuated_joint="${side}_gripper_motor_slider_joint"
                                 simulated_reduction="314.16"   />
     </transmission>
+-->
   </xacro:macro>
 </robot>
